File: KiCAD/DC33/DC33.kicad_pcb (KiCad board)
At the start: 4 copper layers, 198.5 x 104.3 mm, 200 parts, among them J1 SAO, J2 PPTC201LFBN-RC, J3 PPTC201LFBN-RC, J4 282834-3, J5 282834-3, J6 FPC-30, J7 S2B-PH-K-S(LF)(SN), Q1 FDN359BN, Q2 CSD17576Q5B, Q3 CSD17576Q5B, U1 PICO2, U10 PCA9536DRG4, U11 ADG849YKSZ-REEL, U12 ADG849YKSZ-REEL, U13 MCP2558FD-H_SN, U14 ADG849YKSZ-REEL, U15 ADG849YKSZ-REEL, U16 ADG849YKSZ-REEL, U17 ADG849YKSZ-REEL, U18 ADG849YKSZ-REEL, U19 ADG849YKSZ-REEL, U2 TS5A3359DCUR, U20 MAX33046EASA+T, U21 ALM2403QPWPRQ1, U22 TMUX1108PWR, U23 TL431AIDBZR, U24 TMUX1108PWR, U25 TL431AIDBZR, U26 TL431AIDBZR, U27 TPS22810TDBVRQ1, U28 TL431AIDBZR, U29 TCAL9539PWR, U3 TPSM828303ARDSR, U30 TPS22810TDBVRQ1, U31 MCP2518FD, U4 ADR510ARTZ-REEL7, U5 MC3479, U6 LM4040D20IDBZR, U7 ISL21010CFH315Z-T7A, U8 BQ297xy, U9 BQ25895RTW, Y1 20MHz 18pF

Commit message: Initial changes - more to do!
Updated based on the new schematic, removed a bunch of old parts. LOTS of traces need to be redone. Parts are imported. Schematic needs the switch to be matched up to the pins on the footprint. Old board shape still there. More silkscreen removed.
Parts:
- removed C19, C21, C22, C23, C49, C51, C60, C61: 1uF, Capacitor_SMD:C_0603_1608Metric
- removed C50, C52: 0.1uF, Capacitor_SMD:C_0603_1608Metric
- removed R43: 0, Resistor_SMD:R_0603_1608Metric
- removed U22, U24: TMUX1108PWR, Library:SOP65P640X120-16N
- removed U23, U25, U26, U28: TL431AIDBZR, Library:SOT95P237X112-3N
- removed U4: ADR510ARTZ-REEL7, Library:SOT95P237X112-3N
- removed U6: LM4040D20IDBZR, Library:SOT95P237X112-3N
- removed U7: ISL21010CFH315Z-T7A, Library:SOT95P237X112-3N-RENESAS
- added R64: 1k, Resistor_SMD:R_0603_1608Metric, B.Cu at (144.7, 132.4)
- added SW1: SW_SPDT, Switches:450404015514, B.Cu at (106.8, 87.9)
- R19: value 470 -> 2k
- R22: value 240 -> 2k
- R23: footprint Library:RESPACK_4X0603 -> Resistor_SMD:R_0603_1608Metric
- R44: value 0 -> 1k
- R45, R50: value 3.16k -> 2k
- R46: value 100 -> 2k
- R47: value 51.1 -> 1k
- R48: value 1.27k -> 1k
- R49: value 1.87k -> 2k
- R52: value 147 -> 1k
- R53: value 619 -> 2k
- R54: value 3.16k -> 1k
- R55: value 1 -> 2k
- R56: value 196 -> 2.2k
- R57: value 3.16k -> 2.2k
- moved R57 46.5 mm to (144.7, 133.9), turned to 0 degrees
- moved R56 40.0 mm to (141.7, 123.0)
- moved R55 29.6 mm to (129.8, 122.0), turned to 180 degrees
- moved R54 21.9 mm to (129.8, 123.6), turned to 0 degrees
- moved R22 20.9 mm to (137.0, 129.8)
- moved R19 19.5 mm to (137.0, 128.1)
- moved R53 18.2 mm to (129.8, 126.7), turned to 0 degrees
- moved R52 17.3 mm to (129.8, 125.1)
- moved R50 13.7 mm to (132.9, 125.2), turned to 0 degrees
- moved R48 13.7 mm to (137.0, 132.9), turned to 180 degrees
- moved R44 12.5 mm to (141.7, 124.5)
- moved R46 10.9 mm to (133.9, 132.9)
- moved R45 7.48 mm to (140.2, 131.4), turned to 0 degrees
- moved R49 6.96 mm to (132.9, 123.6), turned to 0 degrees
- moved R23 4.14 mm to (139.9, 94.5), turned to 90 degrees
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Connections:
- C25 pad 1: Net-(C25-Pad1) -> Net-(SW1-C)
- J7 pad 1: Net-(C25-Pad1) -> Net-(SW1-B)
- R18 pad 2: GND -> (no net)
- R18 pad 3: GND -> (no net)
- R18 pad 4: GND -> (no net)
- R18 pad 5: /Diff injector/H_V0 -> (no net)
- R18 pad 6: /Diff injector/H_V1 -> (no net)
- R18 pad 7: /Diff injector/H_V2 -> (no net)
- R19 pad 1: /Diff injector/+5V_SW -> Net-(R19-Pad1)
- R19 pad 2: /Diff injector/1V -> GND
- R22 pad 1: /Diff injector/+5V_SW -> Net-(R19-Pad1)
- R22 pad 2: /Diff injector/2V -> /Diff injector/L_V0
- R23 pad 1: GND -> /Diff injector/L_Z0
- R31 pad 2: Net-(C25-Pad1) -> Net-(SW1-C)
- R44 pad 1: Net-(U21-IN(1)-) -> Net-(U21-OUT(2))
- R44 pad 2: Net-(U21-OUT(1)) -> Net-(U21-IN(2)-)
- R45 pad 2: GND -> /Diff injector/L_V1
- R46 pad 1: /Diff injector/+5V_SW -> Net-(U21-IN(2)+)
- R46 pad 2: /Diff injector/3V5 -> /Diff injector/L_V2
- R47 pad 1: /Diff injector/+5V_SW -> Net-(R19-Pad1)
- R47 pad 2: /Diff injector/4V -> Net-(R45-Pad1)
- R48 pad 1: /Diff injector/3V5 -> Net-(R45-Pad1)
- R48 pad 2: Net-(R48-Pad2) -> Net-(U21-IN(2)+)
- R49 pad 1: /Diff injector/4V -> Net-(R49-Pad1)
- R49 pad 2: Net-(R45-Pad1) -> GND
- R50 pad 1: Net-(R48-Pad2) -> Net-(R49-Pad1)
- R50 pad 2: GND -> /Diff injector/H_V0
- R52 pad 1: /Diff injector/+5V_SW -> Net-(R49-Pad1)
- R52 pad 2: /Diff injector/3V -> Net-(R52-Pad2)
- R53 pad 1: /Diff injector/3V -> Net-(R52-Pad2)
- R53 pad 2: Net-(R53-Pad2) -> /Diff injector/H_V1
- R54 pad 1: Net-(R53-Pad2) -> Net-(R52-Pad2)
- R54 pad 2: GND -> Net-(U21-IN(1)+)
- R55 pad 1: /Diff injector/2V5 -> Net-(U21-IN(1)+)
- R55 pad 2: Net-(R55-Pad2) -> /Diff injector/H_V2
- R56 pad 1: /Diff injector/+5V_SW -> GND
- R56 pad 2: /Diff injector/2V5 -> Net-(U21-OUT(2))
- R57 pad 1: Net-(R55-Pad2) -> GND
- R57 pad 2: GND -> Net-(U21-IN(1)-)
- U9 pad 13: Net-(C25-Pad1) -> Net-(SW1-C)
- U9 pad 14: Net-(C25-Pad1) -> Net-(SW1-C)
Routing:
- net /Diff injector/2V5: track 54.0 -> 0.00 mm, vias 2 -> 0
- net /Diff injector/3V: track 43.1 -> 0.00 mm, vias 2 -> 0
- net /Diff injector/2V: track 35.4 -> 0.00 mm, vias 2 -> 0
- net /Diff injector/4V: track 33.6 -> 0.00 mm, vias 2 -> 0
- net /Diff injector/1V: track 32.3 -> 0.00 mm, vias 2 -> 0
- net /Diff injector/3V5: track 31.4 -> 0.00 mm, vias 2 -> 0
- net /Diff injector/1V5: track 28.8 -> 0.00 mm, vias 2 -> 0
- net Net-(C25-Pad1): track 25.1 -> 0.00 mm
- net /TX_DISABLE: track 145.1 -> 120.5 mm
- net /Diff injector/0V: track 17.8 -> 0.00 mm, vias 2 -> 0
- net /Diff injector/+5V_SW: track 58.3 -> 42.0 mm, vias 14 -> 8
- net Net-(SW1-C): track 0.00 -> 15.4 mm
- net Net-(U21-IN(2)+): track 21.8 -> 6.70 mm, vias 4 -> 2
- net /Diff injector/H_V2: track 36.5 -> 25.0 mm
- net /Diff injector/H_V1: track 36.8 -> 26.4 mm
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