File: KiCAD/DC33/power.kicad_sch (KiCad schematic)
At the start: 36 parts, among them J7 S2B-PH-K-S(LF)(SN), Q2 CSD17576Q5B, Q3 CSD17576Q5B, U3 TPSM828303ARDSR, U8 BQ297xy, U9 BQ25895RTW

Commit message: render
Changed lines of the file:
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@@
-	)
-	(junction
-		(at 166.37 72.39)
-		(diameter 0)
-		(color 0 0 0 0)
 	)
 	(junction
@@
 	)
 	(junction
+		(at 166.37 77.47)
+		(diameter 0)
+		(color 0 0 0 0)
+	)
+	(junction
 		(at 171.45 52.07)
 		(diameter 0)
@@
 	(wire
 		(pts
-			(xy 194.31 72.39) (xy 194.31 97.79)
+			(xy 194.31 77.47) (xy 194.31 97.79)
 		)
 		(stroke
@@
 	(wire
 		(pts
+			(xy 166.37 77.47) (xy 194.31 77.47)
+		)
+		(stroke
+			(width 0)
+			(type default)
+		)
+	)
+	(wire
+		(pts
 			(xy 186.69 140.97) (xy 186.69 127)
 		)
@@
 	(wire
 		(pts
-			(xy 137.16 72.39) (xy 166.37 72.39)
+			(xy 137.16 77.47) (xy 166.37 77.47)
 		)
 		(stroke
@@
 	(wire
 		(pts
-			(xy 166.37 72.39) (xy 166.37 86.36)
+			(xy 166.37 77.47) (xy 166.37 86.36)
 		)
 		(stroke
@@
 	(wire
 		(pts
-			(xy 137.16 72.39) (xy 137.16 64.77)
-		)
-		(stroke
-			(width 0)
-			(type default)
-		)
-	)
-	(wire
-		(pts
-			(xy 166.37 72.39) (xy 194.31 72.39)
-		)
-		(stroke
+			(xy 137.16 77.47) (xy 137.16 64.77)
+		)
+		(stroke

Commit message: switch
Parts:
- added SW1: SW_SPDT, symbol Switch:SW_SPDT
Connections:
- net at C25.1, R31.2, U9.13 (BAT)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: now also SW1.3 (C); no longer J7.1
- new net: J7.1, SW1.2 (B)
- no-connect marks 5 -> 6
Changed lines of the file:
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@@
 	)
 	(junction
+		(at 166.37 77.47)
+		(diameter 0)
+		(color 0 0 0 0)
+	)
+	(junction
 		(at 40.64 46.99)
 		(diameter 0)
@@
 	)
 	(junction
-		(at 166.37 77.47)
-		(diameter 0)
-		(color 0 0 0 0)
-	)
-	(junction
 		(at 171.45 52.07)
 		(diameter 0)
@@
 	)
 	(no_connect
+		(at 175.26 82.55)
+	)
+	(no_connect
 		(at 107.95 74.93)
 	)
@@
 	(wire
 		(pts
-			(xy 194.31 77.47) (xy 194.31 97.79)
+			(xy 194.31 80.01) (xy 194.31 97.79)
 		)
 		(stroke
@@
 	(wire
 		(pts
-			(xy 166.37 77.47) (xy 194.31 77.47)
-		)
-		(stroke
-			(width 0)
-			(type default)
-		)
-	)
-	(wire
-		(pts
 			(xy 186.69 140.97) (xy 186.69 127)
 		)
@@
 	(wire
 		(pts
+			(xy 185.42 80.01) (xy 194.31 80.01)
+		)
+		(stroke
+			(width 0)
+			(type default)
+		)
+	)
+	(wire
+		(pts
 			(xy 147.32 121.92) (xy 147.32 140.97)
 		)
@@
 	(wire
 		(pts
+			(xy 175.26 77.47) (xy 166.37 77.47)
+		)
+		(stroke
+			(width 0)
+			(type default)
+		)
+	)
+	(wire
+		(pts
 			(xy 54.61 77.47) (xy 54.61 63.5)
 		)
@@
 					(unit 1)
 				)
+			)
+		)
+	)
+	(symbol
+		(lib_id "Switch:SW_SPDT")
+		(at 180.34 80.01 180)
+		(unit 1)
+		(body_style 1)
+		(exclude_from_sim no)
+		(in_bom yes)
+		(on_board yes)
+		(in_pos_files yes)
+		(dnp no)
+		(fields_autoplaced yes)
+		(property "Reference" "SW1"
+			(at 180.34 71.12 0)
+			(show_name no)
+			(do_not_autoplace no)
+			(effects
+				(font
+					(size 1.27 1.27)
+				)
+			)
+		)
+		(property "Value" "SW_SPDT"
+			(at 180.34 73.66 0)
+			(show_name no)
+			(do_not_autoplace no)
+			(effects
+				(font
+					(size 1.27 1.27)
+				)
+			)
+		)
+		(property "Footprint" ""
+			(at 180.34 80.01 0)
+			(hide yes)
+			(show_name no)
+			(do_not_autoplace no)
+			(effects
+				(font
+					(size 1.27 1.27)
+				)
+			)
+		)
+		(property "Datasheet" ""
+			(at 180.34 72.39 0)
+			(hide yes)
+			(show_name no)
+			(do_not_autoplace no)
+			(effects
+				(font
+					(size 1.27 1.27)
+				)
+			)
+		)
+		(property "Description" "Switch, single pole double throw"
+			(at 180.34 80.01 0)
+			(hide yes)
+			(show_name no)
+			(do_not_autoplace no)
+			(effects
+				(font
+					(size 1.27 1.27)
+				)
+			)
+		)
+		(pin "3"
+		)
+		(pin "2"
+		)
+		(pin "1"
+		)
+		(instances
+			(project "DC33"
+				(path "/c031bbd5-e288-461b-abff-d4e8c5230266/08e3877e-c84c-4b5e-b5b4-7862d19d4233"
+					(reference "SW1")
+					(unit 1)
+				)
