File: KiCAD/DC33/power.kicad_sch (KiCad schematic)
At the start: 36 parts, among them J7 S2B-PH-K-S(LF)(SN), Q2 CSD17576Q5B, Q3 CSD17576Q5B, U3 TPSM828303ARDSR, U8 BQ297xy, U9 BQ25895RTW

Commit message: power switch
Parts:
- added SW1: SW_SPDT, symbol Switch:SW_SPDT
Connections:
- net at C25.1, R31.2, U9.13 (BAT)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: now also SW1.3 (C); no longer J7.1
- new net: J7.1, SW1.2 (B)
Changed lines of the file:
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@@
 	)
 	(junction
-		(at 128.27 140.97)
+		(at 166.37 72.39)
 		(diameter 0)
 		(color 0 0 0 0)
 	)
 	(junction
-		(at 273.05 68.58)
+		(at 128.27 140.97)
 		(diameter 0)
 		(color 0 0 0 0)
 	)
 	(junction
-		(at 166.37 72.39)
+		(at 273.05 68.58)
 		(diameter 0)
 		(color 0 0 0 0)
@@
 	(wire
 		(pts
+			(xy 185.42 74.93) (xy 194.31 74.93)
+		)
+		(stroke
+			(width 0)
+			(type default)
+		)
+	)
+	(wire
+		(pts
 			(xy 198.12 59.69) (xy 198.12 67.31)
 		)
@@
 	(wire
 		(pts
-			(xy 194.31 72.39) (xy 194.31 97.79)
-		)
-		(stroke
-			(width 0)
-			(type default)
-		)
-	)
-	(wire
-		(pts
 			(xy 250.19 52.07) (xy 261.62 52.07)
 		)
@@
 	(wire
 		(pts
+			(xy 194.31 74.93) (xy 194.31 97.79)
+		)
+		(stroke
+			(width 0)
+			(type default)
+		)
+	)
+	(wire
+		(pts
 			(xy 157.48 111.76) (xy 166.37 111.76)
 		)
@@
 	(wire
 		(pts
-			(xy 147.32 121.92) (xy 147.32 140.97)
+			(xy 166.37 72.39) (xy 175.26 72.39)
 		)
 		(stroke
@@
 	(wire
 		(pts
-			(xy 137.16 72.39) (xy 137.16 64.77)
+			(xy 147.32 121.92) (xy 147.32 140.97)
 		)
 		(stroke
@@
 	(wire
 		(pts
-			(xy 166.37 72.39) (xy 194.31 72.39)
+			(xy 137.16 72.39) (xy 137.16 64.77)
 		)
 		(stroke
@@
 		)
 		(instances
-			(project "Untitled"
+			(project "DC33"
 				(path "/c031bbd5-e288-461b-abff-d4e8c5230266/08e3877e-c84c-4b5e-b5b4-7862d19d4233"
 					(reference "#PWR029")
@@
 		)
 		(instances
-			(project "Untitled"
+			(project "DC33"
 				(path "/c031bbd5-e288-461b-abff-d4e8c5230266/08e3877e-c84c-4b5e-b5b4-7862d19d4233"
 					(reference "U8")
@@
 		)
 		(instances
-			(project "Untitled"
+			(project "DC33"
 				(path "/c031bbd5-e288-461b-abff-d4e8c5230266/08e3877e-c84c-4b5e-b5b4-7862d19d4233"
 					(reference "#PWR024")
@@
 		)
 		(instances
-			(project "Untitled"
+			(project "DC33"
 				(path "/c031bbd5-e288-461b-abff-d4e8c5230266/08e3877e-c84c-4b5e-b5b4-7862d19d4233"
 					(reference "R24")
@@
 		)
 		(instances
-			(project "Untitled"
+			(project "DC33"
 				(path "/c031bbd5-e288-461b-abff-d4e8c5230266/08e3877e-c84c-4b5e-b5b4-7862d19d4233"
 					(reference "D1")
@@
 		)
 		(instances
-			(project "Untitled"
+			(project "DC33"
 				(path "/c031bbd5-e288-461b-abff-d4e8c5230266/08e3877e-c84c-4b5e-b5b4-7862d19d4233"
 					(reference "#PWR019")
@@
 		)
 		(instances
-			(project "Untitled"
+			(project "DC33"
 				(path "/c031bbd5-e288-461b-abff-d4e8c5230266/08e3877e-c84c-4b5e-b5b4-7862d19d4233"
 					(reference "#PWR026")
@@
 	)
 	(symbol
+		(lib_id "Switch:SW_SPDT")
+		(at 180.34 74.93 180)
+		(unit 1)
+		(exclude_from_sim no)
+		(in_bom yes)
+		(on_board yes)
+		(dnp no)
+		(fields_autoplaced yes)
+		(property "Reference" "SW1"
+			(at 180.34 66.04 0)
+			(effects
+				(font
+					(size 1.27 1.27)
+				)
+			)
+		)
+		(property "Value" "SW_SPDT"
+			(at 180.34 68.58 0)
+			(effects
+				(font
+					(size 1.27 1.27)
+				)
+			)
+		)
+		(property "Footprint" ""
+			(at 180.34 74.93 0)
+			(effects
+				(font
+					(size 1.27 1.27)
+				)
+				(hide yes)
+			)
+		)
+		(property "Datasheet" "~"
+			(at 180.34 67.31 0)
+			(effects
+				(font
+					(size 1.27 1.27)
+				)
+				(hide yes)
+			)
+		)
+		(property "Description" "Switch, single pole double throw"
+			(at 180.34 74.93 0)
+			(effects
+				(font
+					(size 1.27 1.27)
+				)
+				(hide yes)
+			)
+		)
+		(pin "3"
+		)
+		(pin "1"
+		)
+		(pin "2"
+		)
+		(instances
+			(project "DC33"
+				(path "/c031bbd5-e288-461b-abff-d4e8c5230266/08e3877e-c84c-4b5e-b5b4-7862d19d4233"
+					(reference "SW1")
+					(unit 1)
+				)
+			)
+		)
+	)
+	(symbol
 		(lib_id "Library:TPSM828303ARDSR")
 		(at 204.47 52.07 0)
@@
 		)
 		(instances
-			(project ""
+			(project "DC33"
 				(path "/c031bbd5-e288-461b-abff-d4e8c5230266/08e3877e-c84c-4b5e-b5b4-7862d19d4233"
 					(reference "U3")
@@
 		)
 		(instances
-			(project "Untitled"
+			(project "DC33"
 				(path "/c031bbd5-e288-461b-abff-d4e8c5230266/08e3877e-c84c-4b5e-b5b4-7862d19d4233"
 					(reference "C58")
@@
 		)
 		(instances
-			(project "Untitled"
+			(project "DC33"
 				(path "/c031bbd5-e288-461b-abff-d4e8c5230266/08e3877e-c84c-4b5e-b5b4-7862d19d4233"
 					(reference "#PWR033")
@@
 		)
 		(instances
-			(project "Untitled"
+			(project "DC33"
 				(path "/c031bbd5-e288-461b-abff-d4e8c5230266/08e3877e-c84c-4b5e-b5b4-7862d19d4233"
 					(reference "#PWR027")
@@
 		)
 		(instances
-			(project "Untitled"
+			(project "DC33"
 				(path "/c031bbd5-e288-461b-abff-d4e8c5230266/08e3877e-c84c-4b5e-b5b4-7862d19d4233"
 					(reference "L1")
@@
 		)
 		(instances
-			(project "Untitled"
+			(project "DC33"
 				(path "/c031bbd5-e288-461b-abff-d4e8c5230266/08e3877e-c84c-4b5e-b5b4-7862d19d4233"
 					(reference "#PWR031")
@@
 		)
 		(instances
-			(project "Untitled"
+			(project "DC33"
 				(path "/c031bbd5-e288-461b-abff-d4e8c5230266/08e3877e-c84c-4b5e-b5b4-7862d19d4233"
 					(reference "#PWR030")
@@
 		)
 		(instances
-			(project "Untitled"
+			(project "DC33"
 				(path "/c031bbd5-e288-461b-abff-d4e8c5230266/08e3877e-c84c-4b5e-b5b4-7862d19d4233"
 					(reference "#PWR020")
@@
 		)
 		(instances
-			(project "Untitled"
+			(project "DC33"
 				(path "/c031bbd5-e288-461b-abff-d4e8c5230266/08e3877e-c84c-4b5e-b5b4-7862d19d4233"
 					(reference "C24")
@@
 		)
 		(instances
-			(project "Untitled"
+			(project "DC33"
 				(path "/c031bbd5-e288-461b-abff-d4e8c5230266/08e3877e-c84c-4b5e-b5b4-7862d19d4233"
 					(reference "C53")
@@
 		)
 		(instances
-			(project "Untitled"
+			(project "DC33"
 				(path "/c031bbd5-e288-461b-abff-d4e8c5230266/08e3877e-c84c-4b5e-b5b4-7862d19d4233"
 					(reference "R26")
@@
 		)
 		(instances
-			(project "Untitled"
+			(project "DC33"
 				(path "/c031bbd5-e288-461b-abff-d4e8c5230266/08e3877e-c84c-4b5e-b5b4-7862d19d4233"
 					(reference "#PWR022")
@@
 		)
 		(instances
-			(project "Untitled"
+			(project "DC33"
 				(path "/c031bbd5-e288-461b-abff-d4e8c5230266/08e3877e-c84c-4b5e-b5b4-7862d19d4233"
 					(reference "R29")
@@
 		)
 		(instances
-			(project "Untitled"
+			(project "DC33"
 				(path "/c031bbd5-e288-461b-abff-d4e8c5230266/08e3877e-c84c-4b5e-b5b4-7862d19d4233"
 					(reference "C26")
@@
 		)
 		(instances
-			(project "Untitled"
+			(project "DC33"
 				(path "/c031bbd5-e288-461b-abff-d4e8c5230266/08e3877e-c84c-4b5e-b5b4-7862d19d4233"
 					(reference "C54")
@@
 		)
 		(instances
-			(project "Untitled"
+			(project "DC33"
 				(path "/c031bbd5-e288-461b-abff-d4e8c5230266/08e3877e-c84c-4b5e-b5b4-7862d19d4233"
 					(reference "R27")
@@
 		)
 		(instances
-			(project "Untitled"
+			(project "DC33"
 				(path "/c031bbd5-e288-461b-abff-d4e8c5230266/08e3877e-c84c-4b5e-b5b4-7862d19d4233"
 					(reference "C59")
@@
 		)
 		(instances
-			(project "Untitled"
+			(project "DC33"
 				(path "/c031bbd5-e288-461b-abff-d4e8c5230266/08e3877e-c84c-4b5e-b5b4-7862d19d4233"
 					(reference "R32")
@@
 		)
 		(instances
-			(project "Untitled"
+			(project "DC33"
 				(path "/c031bbd5-e288-461b-abff-d4e8c5230266/08e3877e-c84c-4b5e-b5b4-7862d19d4233"
 					(reference "R30")
@@
 		)
 		(instances
-			(project "Untitled"
+			(project "DC33"
 				(path "/c031bbd5-e288-461b-abff-d4e8c5230266/08e3877e-c84c-4b5e-b5b4-7862d19d4233"
 					(reference "#PWR025")
@@
 		)
 		(instances
-			(project "Untitled"
+			(project "DC33"
 				(path "/c031bbd5-e288-461b-abff-d4e8c5230266/08e3877e-c84c-4b5e-b5b4-7862d19d4233"
 					(reference "R28")
@@
 		)
 		(instances
-			(project "Untitled"
+			(project "DC33"
 				(path "/c031bbd5-e288-461b-abff-d4e8c5230266/08e3877e-c84c-4b5e-b5b4-7862d19d4233"
 					(reference "C25")
@@
 		)
 		(instances
-			(project "Untitled"
+			(project "DC33"
 				(path "/c031bbd5-e288-461b-abff-d4e8c5230266/08e3877e-c84c-4b5e-b5b4-7862d19d4233"
 					(reference "R25")
@@
 		)
 		(instances
-			(project "Untitled"
+			(project "DC33"
 				(path "/c031bbd5-e288-461b-abff-d4e8c5230266/08e3877e-c84c-4b5e-b5b4-7862d19d4233"
 					(reference "#PWR028")
@@
 		)
 		(instances
-			(project "Untitled"
+			(project "DC33"
 				(path "/c031bbd5-e288-461b-abff-d4e8c5230266/08e3877e-c84c-4b5e-b5b4-7862d19d4233"
 					(reference "C27")
@@
 		)
 		(instances
-			(project "Untitled"
+			(project "DC33"
 				(path "/c031bbd5-e288-461b-abff-d4e8c5230266/08e3877e-c84c-4b5e-b5b4-7862d19d4233"
 					(reference "U9")
@@
 		)
 		(instances
-			(project "Untitled"
+			(project "DC33"
 				(path "/c031bbd5-e288-461b-abff-d4e8c5230266/08e3877e-c84c-4b5e-b5b4-7862d19d4233"
 					(reference "C28")
@@
 		)
 		(instances
-			(project "Untitled"
+			(project "DC33"
 				(path "/c031bbd5-e288-461b-abff-d4e8c5230266/08e3877e-c84c-4b5e-b5b4-7862d19d4233"
 					(reference "#PWR023")
@@
 		)
 		(instances
-			(project "Untitled"
+			(project "DC33"
 				(path "/c031bbd5-e288-461b-abff-d4e8c5230266/08e3877e-c84c-4b5e-b5b4-7862d19d4233"
 					(reference "R31")
@@
 		)
 		(instances
-			(project "Untitled"
+			(project "DC33"
 				(path "/c031bbd5-e288-461b-abff-d4e8c5230266/08e3877e-c84c-4b5e-b5b4-7862d19d4233"
 					(reference "#PWR032")
@@
 		)
 		(instances
-			(project "Untitled"
+			(project "DC33"
 				(path "/c031bbd5-e288-461b-abff-d4e8c5230266/08e3877e-c84c-4b5e-b5b4-7862d19d4233"
 					(reference "Q2")
@@
 		)
 		(instances
-			(project "Untitled"
+			(project "DC33"
 				(path "/c031bbd5-e288-461b-abff-d4e8c5230266/08e3877e-c84c-4b5e-b5b4-7862d19d4233"
 					(reference "Q3")
@@
 		)
 		(instances
-			(project "Untitled"
+			(project "DC33"
 				(path "/c031bbd5-e288-461b-abff-d4e8c5230266/08e3877e-c84c-4b5e-b5b4-7862d19d4233"
 					(reference "C55")

Commit message: Initial changes - more to do!
Updated based on the new schematic, removed a bunch of old parts. LOTS of traces need to be redone. Parts are imported. Schematic needs the switch to be matched up to the pins on the footprint. Old board shape still there. More silkscreen removed.
Parts:
- SW1: footprint (none) -> Switches:450404015514
Other:
- note added: "TODO: match pins to footprint or change schematic part to match footprint"
